Commit message: Change material color from silver to green

File: Universal_Robots_ROS2_Tutorials/my_robot_cell/my_robot_cell_description/urdf/simrobot_my_robot_cell_macro.xacro (robot description, xacro)
@@ -116,5 +116,7 @@
           <mesh filename="file:////home/cem/colcon_ws/src/Universal_Robots_ROS2_Description/meshes/ur10e/collision/conveyorbelt.stl" scale="0.001 0.001 0.001"/>
         </geometry>
-        <material name="silver"/>
+        <material name="green">
+          <color rgba="0 1 0 1"/>
+        </material>
       </visual>
       <collision>
