Commit message: Add files via upload

File: Universal_Robots_ROS2_Tutorials/my_robot_cell/my_robot_cell_description/urdf/my_robot_cell_macro.xacro (robot description, xacro)
@@ -14,4 +14,5 @@
     use_fake_hardware:=false
     tf_prefix:='ur10e_'
+    use_gripper:=false
     ">
     <!-- no prefix for real robot, robot1_ for sim -->
@@ -31,12 +32,12 @@
         <origin rpy="0 0 0" xyz="0 0 0"/>
         <geometry>
-          <mesh filename="file:////home/cem/colcon_ws/src/Universal_Robots_ROS2_Description/meshes/ur10e/collision/base_link.stl" scale="0.001 0.001 0.001"/>
-        </geometry>
-        <material name="silver"/>
-      </visual>
-      <collision>
-        <origin rpy="0 0 0" xyz="0 0 0"/>
-        <geometry>
-          <mesh filename="file:////home/cem/colcon_ws/src/Universal_Robots_ROS2_Description/meshes/ur10e/collision/base_link.stl" scale="0.001 0.001 0.001"/>
+          <mesh filename="file:////home/emirhan/colcon_ws/src/Universal_Robots_ROS2_Description/meshes/ur10e/collision/base_link.stl" scale="0.001 0.001 0.001"/>
+        </geometry>
+        <material name="silver"/>
+      </visual>
+      <collision>
+        <origin rpy="0 0 0" xyz="0 0 0"/>
+        <geometry>
+          <mesh filename="file:////home/emirhan/colcon_ws/src/Universal_Robots_ROS2_Description/meshes/ur10e/collision/base_link.stl" scale="0.001 0.001 0.001"/>
         </geometry>
       </collision>
@@ -57,5 +58,5 @@
         <origin xyz="0 0 0" rpy="0 0 0"/>
         <geometry>
-          <mesh filename="file:////home/cem/colcon_ws/src/Universal_Robots_ROS2_Description/meshes/ur10e/collision/chassis.stl" scale="0.001 0.001 0.001"/>
+          <mesh filename="file:////home/emirhan/colcon_ws/src/Universal_Robots_ROS2_Description/meshes/ur10e/collision/chassis.stl" scale="0.001 0.001 0.001"/>
         </geometry>
         <material name="chassis_material">
@@ -66,5 +67,5 @@
         <origin xyz="0 0 0" rpy="0 0 0"/>
         <geometry>
-          <mesh filename="file:////home/cem/colcon_ws/src/Universal_Robots_ROS2_Description/meshes/ur10e/collision/chassis.stl" scale="0.001 0.001 0.001"/>
+          <mesh filename="file:////home/emirhan/colcon_ws/src/Universal_Robots_ROS2_Description/meshes/ur10e/collision/chassis.stl" scale="0.001 0.001 0.001"/>
         </geometry>
       </collision>
@@ -79,5 +80,5 @@
         <origin rpy="0 0 0" xyz="0.158 -0.115 -0.58635"/>
         <geometry>
-          <mesh filename="file:////home/cem/colcon_ws/src/Universal_Robots_ROS2_Description/meshes/ur10e/collision/linear_axis_moving_link.stl" scale="0.001 0.001 0.001"/>
+          <mesh filename="file:////home/emirhan/colcon_ws/src/Universal_Robots_ROS2_Description/meshes/ur10e/collision/linear_axis_moving_link.stl" scale="0.001 0.001 0.001"/>
         </geometry>
         <material name="silver"/>
@@ -86,5 +87,5 @@
         <origin rpy="0 0 0" xyz="0.158 -0.115 -0.58635"/>
         <geometry>
-          <mesh filename="file:////home/cem/colcon_ws/src/Universal_Robots_ROS2_Description/meshes/ur10e/collision/linear_axis_moving_link.stl" scale="0.001 0.001 0.001"/>
+          <mesh filename="file:////home/emirhan/colcon_ws/src/Universal_Robots_ROS2_Description/meshes/ur10e/collision/linear_axis_moving_link.stl" scale="0.001 0.001 0.001"/>
         </geometry>
       </collision>
@@ -99,12 +100,12 @@
         <origin rpy="0 0 0" xyz="0 0 0"/>
         <geometry>
-          <mesh filename="file:////home/cem/colcon_ws/src/Universal_Robots_ROS2_Description/meshes/ur10e/collision/wall_door.stl" scale="0.001 0.001 0.001"/>
-        </geometry>
-        <material name="silver"/>
-      </visual>
-      <collision>
-        <origin rpy="0 0 0" xyz="0 0 0"/>
-        <geometry>
-          <mesh filename="file:////home/cem/colcon_ws/src/Universal_Robots_ROS2_Description/meshes/ur10e/collision/wall_door.stl" scale="0.001 0.001 0.001"/>
+          <mesh filename="file:////home/emirhan/colcon_ws/src/Universal_Robots_ROS2_Description/meshes/ur10e/collision/wall_door.stl" scale="0.001 0.001 0.001"/>
+        </geometry>
+        <material name="silver"/>
+      </visual>
+      <collision>
+        <origin rpy="0 0 0" xyz="0 0 0"/>
+        <geometry>
+          <mesh filename="file:////home/emirhan/colcon_ws/src/Universal_Robots_ROS2_Description/meshes/ur10e/collision/wall_door.stl" scale="0.001 0.001 0.001"/>
         </geometry>
       </collision>
@@ -119,12 +120,12 @@
         <origin rpy="0 0 0" xyz="0 0 0"/>
         <geometry>
-          <mesh filename="file:////home/cem/colcon_ws/src/Universal_Robots_ROS2_Description/meshes/ur10e/collision/wall_server.stl" scale="0.001 0.001 0.001"/>
-        </geometry>
-        <material name="silver"/>
-      </visual>
-      <collision>
-        <origin rpy="0 0 0" xyz="0 0 0"/>
-        <geometry>
-          <mesh filename="file:////home/cem/colcon_ws/src/Universal_Robots_ROS2_Description/meshes/ur10e/collision/wall_server.stl" scale="0.001 0.001 0.001"/>
+          <mesh filename="file:////home/emirhan/colcon_ws/src/Universal_Robots_ROS2_Description/meshes/ur10e/collision/wall_server.stl" scale="0.001 0.001 0.001"/>
+        </geometry>
+        <material name="silver"/>
+      </visual>
+      <collision>
+        <origin rpy="0 0 0" xyz="0 0 0"/>
+        <geometry>
+          <mesh filename="file:////home/emirhan/colcon_ws/src/Universal_Robots_ROS2_Description/meshes/ur10e/collision/wall_server.stl" scale="0.001 0.001 0.001"/>
         </geometry>
       </collision>
@@ -139,12 +140,12 @@
         <origin rpy="0 0 0" xyz="0 0 0"/>
         <geometry>
-          <mesh filename="file:////home/cem/colcon_ws/src/Universal_Robots_ROS2_Description/meshes/ur10e/collision/alumuniumtable.stl" scale="0.001 0.001 0.001"/>
-        </geometry>
-        <material name="silver"/>
-      </visual>
-      <collision>
-        <origin rpy="0 0 0" xyz="0 0 0"/>
-        <geometry>
-          <mesh filename="file:////home/cem/colcon_ws/src/Universal_Robots_ROS2_Description/meshes/ur10e/collision/alumuniumtable.stl" scale="0.001 0.001 0.001"/>
+          <mesh filename="file:////home/emirhan/colcon_ws/src/Universal_Robots_ROS2_Description/meshes/ur10e/collision/alumuniumtable.stl" scale="0.001 0.001 0.001"/>
+        </geometry>
+        <material name="silver"/>
+      </visual>
+      <collision>
+        <origin rpy="0 0 0" xyz="0 0 0"/>
+        <geometry>
+          <mesh filename="file:////home/emirhan/colcon_ws/src/Universal_Robots_ROS2_Description/meshes/ur10e/collision/alumuniumtable.stl" scale="0.001 0.001 0.001"/>
         </geometry>
       </collision>
@@ -159,12 +160,12 @@
         <origin rpy="0 0 0" xyz="0 0 0"/>
         <geometry>
-          <mesh filename="file:////home/cem/colcon_ws/src/Universal_Robots_ROS2_Description/meshes/ur10e/collision/conveyorbelt.stl" scale="0.001 0.001 0.001"/>
-        </geometry>
-        <material name="silver"/>
-      </visual>
-      <collision>
-        <origin rpy="0 0 0" xyz="0 0 0"/>
-        <geometry>
-          <mesh filename="file:////home/cem/colcon_ws/src/Universal_Robots_ROS2_Description/meshes/ur10e/collision/conveyorbelt.stl" scale="0.001 0.001 0.001"/>
+          <mesh filename="file:////home/emirhan/colcon_ws/src/Universal_Robots_ROS2_Description/meshes/ur10e/collision/conveyorbelt.stl" scale="0.001 0.001 0.001"/>
+        </geometry>
+        <material name="silver"/>
+      </visual>
+      <collision>
+        <origin rpy="0 0 0" xyz="0 0 0"/>
+        <geometry>
+          <mesh filename="file:////home/emirhan/colcon_ws/src/Universal_Robots_ROS2_Description/meshes/ur10e/collision/conveyorbelt.stl" scale="0.001 0.001 0.001"/>
         </geometry>
       </collision>
@@ -185,12 +186,12 @@
         <origin xyz="0 0 0" rpy="0 0 0"/>
         <geometry>
-          <mesh filename="file:////home/cem/colcon_ws/src/Universal_Robots_ROS2_Description/meshes/ur10e/collision/stackable_bin.stl" scale="0.001 0.001 0.001"/>
-        </geometry>
-        <material name="silver"/>
-      </visual>
-      <collision>
-        <origin xyz="0 0 0" rpy="0 0 0"/>
-        <geometry>
-          <mesh filename="file:////home/cem/colcon_ws/src/Universal_Robots_ROS2_Description/meshes/ur10e/collision/stackable_bin.stl" scale="0.001 0.001 0.001"/>
+          <mesh filename="file:////home/emirhan/colcon_ws/src/Universal_Robots_ROS2_Description/meshes/ur10e/collision/stackable_bin.stl" scale="0.001 0.001 0.001"/>
+        </geometry>
+        <material name="silver"/>
+      </visual>
+      <collision>
+        <origin xyz="0 0 0" rpy="0 0 0"/>
+        <geometry>
+          <mesh filename="file:////home/emirhan/colcon_ws/src/Universal_Robots_ROS2_Description/meshes/ur10e/collision/stackable_bin.stl" scale="0.001 0.001 0.001"/>
         </geometry>
       </collision>
@@ -284,4 +285,5 @@
       generate_ros2_control_tag="false"
       sim_ignition="${sim_ignition}"
+      use_gripper="${use_gripper}"
     >
       <origin xyz="0 0 0" rpy="0 0 0" />
