Commit message: IMX Optical frame

File: Universal_Robots_ROS2_Description/urdf/simrobot_ur_macro.xacro (robot description, xacro)
@@ -139,5 +139,5 @@
         <origin xyz="0.105561 -0.1918 -0.6445" rpy="0 0 0"/>
         <geometry>
-          <mesh filename="file:////home/cem/colcon_ws/src/Universal_Robots_ROS2_Description/meshes/ur10e/secondrobotvisual/base.stl" scale="0.001 0.001 0.001"/>
+          <mesh filename="file:////home/emirhan/colcon_ws/src/Universal_Robots_ROS2_Description/meshes/ur10e/secondrobotvisual/base.stl" scale="0.001 0.001 0.001"/>
         </geometry>
         <material name="silver"/>
@@ -146,5 +146,5 @@
         <origin xyz="0.105561 -0.1918 -0.6445" rpy="0 0 0"/>
         <geometry>
-          <mesh filename="file:////home/cem/colcon_ws/src/Universal_Robots_ROS2_Description/meshes/ur10e/secondrobotcollision/base.stl" scale="0.001 0.001 0.001"/>
+          <mesh filename="file:////home/emirhan/colcon_ws/src/Universal_Robots_ROS2_Description/meshes/ur10e/secondrobotcollision/base.stl" scale="0.001 0.001 0.001"/>
         </geometry>
         <material name="silver"/>
@@ -158,5 +158,5 @@
         <origin xyz="0.105565 -0.1918 -0.74405" rpy="0 0 0"/>
         <geometry>
-          <mesh filename="file:////home/cem/colcon_ws/src/Universal_Robots_ROS2_Description/meshes/ur10e/secondrobotvisual/shoulder.stl" scale="0.001 0.001 0.001"/>
+          <mesh filename="file:////home/emirhan/colcon_ws/src/Universal_Robots_ROS2_Description/meshes/ur10e/secondrobotvisual/shoulder.stl" scale="0.001 0.001 0.001"/>
         </geometry>
         <material name="silver"/>
@@ -165,5 +165,5 @@
         <origin xyz="0.105565 -0.1918 -0.74405" rpy="0 0 0"/>
         <geometry>
-          <mesh filename="file:////home/cem/colcon_ws/src/Universal_Robots_ROS2_Description/meshes/ur10e/secondrobotcollision/shoulder.stl" scale="0.001 0.001 0.001"/>
+          <mesh filename="file:////home/emirhan/colcon_ws/src/Universal_Robots_ROS2_Description/meshes/ur10e/secondrobotcollision/shoulder.stl" scale="0.001 0.001 0.001"/>
         </geometry>
       </collision>
@@ -185,5 +185,5 @@
         <origin xyz="0.105565 -0.2778 -0.83405" rpy="0 0 0"/>
         <geometry>
-          <mesh filename="file:////home/cem/colcon_ws/src/Universal_Robots_ROS2_Description/meshes/ur10e/secondrobotvisual/upperarm.stl" scale="0.001 0.001 0.001"/>
+          <mesh filename="file:////home/emirhan/colcon_ws/src/Universal_Robots_ROS2_Description/meshes/ur10e/secondrobotvisual/upperarm.stl" scale="0.001 0.001 0.001"/>
         </geometry>
         <material name="silver"/>
@@ -192,5 +192,5 @@
         <origin xyz="0.105565 -0.2778 -0.83405" rpy="0 0 0"/>
         <geometry>
-          <mesh filename="file:////home/cem/colcon_ws/src/Universal_Robots_ROS2_Description/meshes/ur10e/secondrobotcollision/upperarm.stl" scale="0.001 0.001 0.001"/>
+          <mesh filename="file:////home/emirhan/colcon_ws/src/Universal_Robots_ROS2_Description/meshes/ur10e/secondrobotcollision/upperarm.stl" scale="0.001 0.001 0.001"/>
         </geometry>
       </collision>
@@ -212,5 +212,5 @@
         <origin xyz="-0.506534 -0.299691 -0.833449" rpy="0 0 0"/>
         <geometry>
-          <mesh filename="file:////home/cem/colcon_ws/src/Universal_Robots_ROS2_Description/meshes/ur10e/secondrobotvisual/forearm.stl" scale="0.001 0.001 0.001"/>
+          <mesh filename="file:////home/emirhan/colcon_ws/src/Universal_Robots_ROS2_Description/meshes/ur10e/secondrobotvisual/forearm.stl" scale="0.001 0.001 0.001"/>
         </geometry>
         <material name="silver"/>
@@ -219,5 +219,5 @@
         <origin xyz="-0.506534 -0.299691 -0.833449" rpy="0 0 0"/>
         <geometry>
-          <mesh filename="file:////home/cem/colcon_ws/src/Universal_Robots_ROS2_Description/meshes/ur10e/secondrobotcollision/forearm.stl" scale="0.001 0.001 0.001"/>
+          <mesh filename="file:////home/emirhan/colcon_ws/src/Universal_Robots_ROS2_Description/meshes/ur10e/secondrobotcollision/forearm.stl" scale="0.001 0.001 0.001"/>
         </geometry>
       </collision>
@@ -239,5 +239,5 @@
       	<origin xyz="-1.078132 -0.301691 -0.833449" rpy="0 0 0"/>
         <geometry>
-          <mesh filename="file:////home/cem/colcon_ws/src/Universal_Robots_ROS2_Description/meshes/ur10e/secondrobotvisual/wrist1.stl" scale="0.001 0.001 0.001"/>
+          <mesh filename="file:////home/emirhan/colcon_ws/src/Universal_Robots_ROS2_Description/meshes/ur10e/secondrobotvisual/wrist1.stl" scale="0.001 0.001 0.001"/>
         </geometry>
         <material name="silver"/>
@@ -246,5 +246,5 @@
         <origin xyz="-1.078132 -0.301691 -0.833449" rpy="0 0 0"/>
         <geometry>
-          <mesh filename="file:////home/cem/colcon_ws/src/Universal_Robots_ROS2_Description/meshes/ur10e/secondrobotcollision/wrist1.stl" scale="0.001 0.001 0.001"/>
+          <mesh filename="file:////home/emirhan/colcon_ws/src/Universal_Robots_ROS2_Description/meshes/ur10e/secondrobotcollision/wrist1.stl" scale="0.001 0.001 0.001"/>
         </geometry>
       </collision>
@@ -266,5 +266,5 @@
         <origin xyz="-1.078132 -0.355691 -0.77175" rpy="0 0 0"/>
         <geometry>
-          <mesh filename="file:////home/cem/colcon_ws/src/Universal_Robots_ROS2_Description/meshes/ur10e/secondrobotvisual/wrist2.stl" scale="0.001 0.001 0.001"/>
+          <mesh filename="file:////home/emirhan/colcon_ws/src/Universal_Robots_ROS2_Description/meshes/ur10e/secondrobotvisual/wrist2.stl" scale="0.001 0.001 0.001"/>
         </geometry>
         <material name="silver"/>
@@ -273,5 +273,5 @@
         <origin xyz="-1.078132 -0.355691 -0.77175" rpy="0 0 0"/>
         <geometry>
-          <mesh filename="file:////home/cem/colcon_ws/src/Universal_Robots_ROS2_Description/meshes/ur10e/secondrobotcollision/wrist2.stl" scale="0.001 0.001 0.001"/>
+          <mesh filename="file:////home/emirhan/colcon_ws/src/Universal_Robots_ROS2_Description/meshes/ur10e/secondrobotcollision/wrist2.stl" scale="0.001 0.001 0.001"/>
         </geometry>
       </collision>
@@ -293,5 +293,5 @@
         <origin xyz="-1.078132 -0.417389 -0.71775" rpy="0 0 0"/>
         <geometry>
-          <mesh filename="file:////home/cem/colcon_ws/src/Universal_Robots_ROS2_Description/meshes/ur10e/secondrobotvisual/wrist3.stl" scale="0.001 0.001 0.001"/>
+          <mesh filename="file:////home/emirhan/colcon_ws/src/Universal_Robots_ROS2_Description/meshes/ur10e/secondrobotvisual/wrist3.stl" scale="0.001 0.001 0.001"/>
         </geometry>
         <material name="silver"/>
@@ -300,5 +300,5 @@
         <origin xyz="-1.078132 -0.417389 -0.71775" rpy="0 0 0"/>
         <geometry>
-          <mesh filename="file:////home/cem/colcon_ws/src/Universal_Robots_ROS2_Description/meshes/ur10e/secondrobotcollision/wrist3.stl" scale="0.001 0.001 0.001"/>
+          <mesh filename="file:////home/emirhan/colcon_ws/src/Universal_Robots_ROS2_Description/meshes/ur10e/secondrobotcollision/wrist3.stl" scale="0.001 0.001 0.001"/>
         </geometry>
       </collision>
@@ -441,5 +441,5 @@
         <origin xyz="-1.106132 -0.502789 -0.727752" rpy="0 0 0"/>
         <geometry>
-          <mesh filename="file:////home/cem/colcon_ws/src/Universal_Robots_ROS2_Description/meshes/ur10e/secondrobotcollision/flange.stl" scale="0.001 0.001 0.001"/>
+          <mesh filename="file:////home/emirhan/colcon_ws/src/Universal_Robots_ROS2_Description/meshes/ur10e/secondrobotcollision/flange.stl" scale="0.001 0.001 0.001"/>
         </geometry>
         <material name="silver"/>
@@ -448,5 +448,5 @@
         <origin xyz="-1.106132 -0.502789 -0.727752" rpy="0 0 0"/>
         <geometry>
-          <mesh filename="file:////home/cem/colcon_ws/src/Universal_Robots_ROS2_Description/meshes/ur10e/secondrobotcollision/flange.stl" scale="0.001 0.001 0.001"/>
+          <mesh filename="file:////home/emirhan/colcon_ws/src/Universal_Robots_ROS2_Description/meshes/ur10e/secondrobotcollision/flange.stl" scale="0.001 0.001 0.001"/>
         </geometry>
       </collision>
@@ -467,5 +467,5 @@
         <origin xyz="-1.078132 -0.477889 -0.717752" rpy="0 0 0"/>
         <geometry>
-          <mesh filename="file:////home/cem/colcon_ws/src/Universal_Robots_ROS2_Description/meshes/ur10e/secondrobotcollision/tool0.stl" scale="0.001 0.001 0.001"/>
+          <mesh filename="file:////home/emirhan/colcon_ws/src/Universal_Robots_ROS2_Description/meshes/ur10e/secondrobotcollision/tool0.stl" scale="0.001 0.001 0.001"/>
         </geometry>
         <material name="silver"/>
@@ -474,5 +474,5 @@
         <origin xyz="-1.078132 -0.477889 -0.717752" rpy="0 0 0"/>
         <geometry>
-          <mesh filename="file:////home/cem/colcon_ws/src/Universal_Robots_ROS2_Description/meshes/ur10e/secondrobotcollision/tool0.stl" scale="0.001 0.001 0.001"/>
+          <mesh filename="file:////home/emirhan/colcon_ws/src/Universal_Robots_ROS2_Description/meshes/ur10e/secondrobotcollision/tool0.stl" scale="0.001 0.001 0.001"/>
         </geometry>
       </collision>
@@ -487,5 +487,5 @@
         <origin xyz="-1.02433 -0.5466 -0.730752" rpy="0 0 0"/>
         <geometry>
-          <mesh filename="file:////home/cem/colcon_ws/src/Universal_Robots_ROS2_Description/meshes/ur10e/secondrobotcollision/sick_camera_mo.stl" scale="0.001 0.001 0.001"/>
+          <mesh filename="file:////home/emirhan/colcon_ws/src/Universal_Robots_ROS2_Description/meshes/ur10e/secondrobotcollision/sick_camera_mo.stl" scale="0.001 0.001 0.001"/>
         </geometry>
         <material name="silver"/>
@@ -494,5 +494,5 @@
         <origin xyz="-1.02433 -0.5466 -0.730752" rpy="0 0 0"/>
         <geometry>
-          <mesh filename="file:////home/cem/colcon_ws/src/Universal_Robots_ROS2_Description/meshes/ur10e/secondrobotcollision/sick_camera_mo.stl" scale="0.001 0.001 0.001"/>
+          <mesh filename="file:////home/emirhan/colcon_ws/src/Universal_Robots_ROS2_Description/meshes/ur10e/secondrobotcollision/sick_camera_mo.stl" scale="0.001 0.001 0.001"/>
         </geometry>
       </collision>
@@ -528,5 +528,5 @@
           <origin xyz="-1.123708 -0.518786 -0.735428" rpy="0 0 0"/>
           <geometry>
-            <mesh filename="file:////home/cem/colcon_ws/src/Universal_Robots_ROS2_Description/meshes/ur10e/secondrobotcollision/gripper_body_1.stl" scale="0.001 0.001 0.001"/>
+            <mesh filename="file:////home/emirhan/colcon_ws/src/Universal_Robots_ROS2_Description/meshes/ur10e/secondrobotcollision/gripper_body_1.stl" scale="0.001 0.001 0.001"/>
           </geometry>
           <material name="violet">
@@ -537,5 +537,5 @@
           <origin xyz="-1.123708 -0.518786 -0.735428" rpy="0 0 0"/>
           <geometry>
-            <mesh filename="file:////home/cem/colcon_ws/src/Universal_Robots_ROS2_Description/meshes/ur10e/secondrobotcollision/gripper_body_1.stl" scale="0.001 0.001 0.001"/>
+            <mesh filename="file:////home/emirhan/colcon_ws/src/Universal_Robots_ROS2_Description/meshes/ur10e/secondrobotcollision/gripper_body_1.stl" scale="0.001 0.001 0.001"/>
           </geometry>
         </collision>
@@ -550,5 +550,5 @@
           <origin xyz="-1.22001 -0.579787 -0.7675" rpy="0 0 0"/>
           <geometry>
-            <mesh filename="file:////home/cem/colcon_ws/src/Universal_Robots_ROS2_Description/meshes/ur10e/secondrobotcollision/gripper_upper_1.stl" scale="0.001 0.001 0.001"/>
+            <mesh filename="file:////home/emirhan/colcon_ws/src/Universal_Robots_ROS2_Description/meshes/ur10e/secondrobotcollision/gripper_upper_1.stl" scale="0.001 0.001 0.001"/>
           </geometry>
           <material name="grey">
@@ -559,5 +559,5 @@
           <origin xyz="-1.22001 -0.579787 -0.7675" rpy="0 0 0"/>
           <geometry>
-            <mesh filename="file:////home/cem/colcon_ws/src/Universal_Robots_ROS2_Description/meshes/ur10e/secondrobotcollision/gripper_upper_1.stl" scale="0.001 0.001 0.001"/>
+            <mesh filename="file:////home/emirhan/colcon_ws/src/Universal_Robots_ROS2_Description/meshes/ur10e/secondrobotcollision/gripper_upper_1.stl" scale="0.001 0.001 0.001"/>
           </geometry>
         </collision>
@@ -572,5 +572,5 @@
           <origin xyz="-1.22001 -0.579787 -0.668" rpy="0 0 0"/>
           <geometry>
-            <mesh filename="file:////home/cem/colcon_ws/src/Universal_Robots_ROS2_Description/meshes/ur10e/secondrobotcollision/gripper_lower_1.stl" scale="0.001 0.001 0.001"/>
+            <mesh filename="file:////home/emirhan/colcon_ws/src/Universal_Robots_ROS2_Description/meshes/ur10e/secondrobotcollision/gripper_lower_1.stl" scale="0.001 0.001 0.001"/>
           </geometry>
           <material name="grey">
@@ -581,5 +581,5 @@
           <origin xyz="-1.22001 -0.579787 -0.668" rpy="0 0 0"/>
           <geometry>
-            <mesh filename="file:////home/cem/colcon_ws/src/Universal_Robots_ROS2_Description/meshes/ur10e/secondrobotcollision/gripper_lower_1.stl" scale="0.001 0.001 0.001"/>
+            <mesh filename="file:////home/emirhan/colcon_ws/src/Universal_Robots_ROS2_Description/meshes/ur10e/secondrobotcollision/gripper_lower_1.stl" scale="0.001 0.001 0.001"/>
           </geometry>
         </collision>
@@ -616,5 +616,5 @@
           <origin xyz="-0.965545 -0.534467 -0.764722" rpy="0 0 0"/>
           <geometry>
-            <mesh filename="file:////home/cem/colcon_ws/src/Universal_Robots_ROS2_Description/meshes/ur10e/secondrobotcollision/IMX_Camera.stl" scale="0.001 0.001 0.001"/>
+            <mesh filename="file:////home/emirhan/colcon_ws/src/Universal_Robots_ROS2_Description/meshes/ur10e/secondrobotcollision/IMX_Camera.stl" scale="0.001 0.001 0.001"/>
           </geometry>
           <material name="silver"/>
@@ -623,5 +623,5 @@
           <origin xyz="-0.965545 -0.534467 -0.764722" rpy="0 0 0"/>
           <geometry>
-            <mesh filename="file:////home/cem/colcon_ws/src/Universal_Robots_ROS2_Description/meshes/ur10e/secondrobotcollision/IMX_Camera.stl" scale="0.001 0.001 0.001"/>
+            <mesh filename="file:////home/emirhan/colcon_ws/src/Universal_Robots_ROS2_Description/meshes/ur10e/secondrobotcollision/IMX_Camera.stl" scale="0.001 0.001 0.001"/>
           </geometry>
         </collision>
@@ -638,4 +638,10 @@
         <parent link="${tf_prefix}IMX_Camera" />
         <child link="${tf_prefix}IMX_Camera_frame_link"/>
+      </joint>
+      <link name="${tf_prefix}IMX_optical_frame"/>
+      <joint name="${tf_prefix}IMX_optical_joint" type="fixed">
+        <origin xyz="0 0 0" rpy="0 0 ${M_PI/2}" />
+        <parent link="${tf_prefix}IMX_Camera_frame_link" />
+        <child link="${tf_prefix}IMX_optical_frame"/>
       </joint>
       <gazebo reference="${tf_prefix}IMX_Camera_frame_link">
@@ -671,5 +677,5 @@
         <origin xyz="-1.078132 -0.537789 -0.707752" rpy="0 0 0"/>
         <geometry>
-          <mesh filename="file:////home/cem/colcon_ws/src/Universal_Robots_ROS2_Description/meshes/ur10e/secondrobotcollision/cable_channel_flange.stl" scale="0.001 0.001 0.001"/>
+          <mesh filename="file:////home/emirhan/colcon_ws/src/Universal_Robots_ROS2_Description/meshes/ur10e/secondrobotcollision/cable_channel_flange.stl" scale="0.001 0.001 0.001"/>
         </geometry>
         <material name="silver"/>
@@ -678,5 +684,5 @@
         <origin xyz="-1.078132 -0.537789 -0.707752" rpy="0 0 0"/>
         <geometry>
-          <mesh filename="file:////home/cem/colcon_ws/src/Universal_Robots_ROS2_Description/meshes/ur10e/secondrobotcollision/cable_channel_flange.stl" scale="0.001 0.001 0.001"/>
+          <mesh filename="file:////home/emirhan/colcon_ws/src/Universal_Robots_ROS2_Description/meshes/ur10e/secondrobotcollision/cable_channel_flange.stl" scale="0.001 0.001 0.001"/>
         </geometry>
       </collision>
@@ -691,5 +697,5 @@
         <origin xyz="-1.078132 -0.486789 -0.669752" rpy="0 0 0"/>
         <geometry>
-          <mesh filename="file:////home/cem/colcon_ws/src/Universal_Robots_ROS2_Description/meshes/ur10e/secondrobotcollision/cable_channel.stl" scale="0.001 0.001 0.001"/>
+          <mesh filename="file:////home/emirhan/colcon_ws/src/Universal_Robots_ROS2_Description/meshes/ur10e/secondrobotcollision/cable_channel.stl" scale="0.001 0.001 0.001"/>
         </geometry>
         <material name="silver"/>
@@ -698,5 +704,5 @@
         <origin xyz="-1.078132 -0.486789 -0.669752" rpy="0 0 0"/>
         <geometry>
-          <mesh filename="file:////home/cem/colcon_ws/src/Universal_Robots_ROS2_Description/meshes/ur10e/secondrobotcollision/cable_channel.stl" scale="0.001 0.001 0.001"/>
+          <mesh filename="file:////home/emirhan/colcon_ws/src/Universal_Robots_ROS2_Description/meshes/ur10e/secondrobotcollision/cable_channel.stl" scale="0.001 0.001 0.001"/>
         </geometry>
       </collision>
