Commit message: Add files via upload

File: Universal_Robots_ROS2_Description/urdf/ur.ros2_control.xacro (robot description, xacro)
@@ -21,4 +21,5 @@
     non_blocking_read:=true
     keep_alive_count:=2
+    use_gripper:=false
     ">
     <ros2_control name="${name}" type="system">
@@ -338,4 +339,22 @@
         </gpio>
       </xacro:unless>
+      <xacro:if value="${use_gripper}">
+        <joint name="${tf_prefix}gripper_joint">
+          <command_interface name="position"/>
+          <state_interface name="position">
+            <param name="initial_value">0.0005</param>
+          </state_interface>
+          <state_interface name="velocity"/>
+          <state_interface name="effort"/>
+        </joint>
+        <joint name="${tf_prefix}gripper_lower_finger_joint">
+          <param name="mimic">${tf_prefix}gripper_joint</param>
+          <param name="multiplier">-1</param>
+          <command_interface name="position"/>
+          <state_interface name="position"/>
+          <state_interface name="velocity"/>
+          <state_interface name="effort"/>
+        </joint>
+      </xacro:if>
     </ros2_control>
   </xacro:macro>

File: Universal_Robots_ROS2_Description/urdf/ur_macro.xacro (robot description, xacro)
@@ -84,5 +84,6 @@
     trajectory_port:=50003
     non_blocking_read:=true
-    keep_alive_count:=2"
+    keep_alive_count:=2
+    use_gripper:=false"
     >
     <!-- Load configuration data from the provided .yaml files -->
@@ -127,4 +128,5 @@
         non_blocking_read="${non_blocking_read}"
         keep_alive_count="${keep_alive_count}"
+        use_gripper="${use_gripper}"
         />
     </xacro:if>
@@ -138,5 +140,5 @@
         <origin xyz="0.105561 -0.1918 -0.6445" rpy="0 0 0"/>
         <geometry>
-          <mesh filename="file:////home/cem/colcon_ws/src/Universal_Robots_ROS2_Description/meshes/ur10e/visual/base.stl" scale="0.001 0.001 0.001"/>
+          <mesh filename="file:////home/emirhan/colcon_ws/src/Universal_Robots_ROS2_Description/meshes/ur10e/visual/base.stl" scale="0.001 0.001 0.001"/>
         </geometry>
         <material name="silver"/>
@@ -145,5 +147,5 @@
         <origin xyz="0.105561 -0.1918 -0.6445" rpy="0 0 0"/>
         <geometry>
-          <mesh filename="file:////home/cem/colcon_ws/src/Universal_Robots_ROS2_Description/meshes/ur10e/collision/base.stl" scale="0.001 0.001 0.001"/>
+          <mesh filename="file:////home/emirhan/colcon_ws/src/Universal_Robots_ROS2_Description/meshes/ur10e/collision/base.stl" scale="0.001 0.001 0.001"/>
         </geometry>
         <material name="silver"/>
@@ -157,5 +159,5 @@
         <origin xyz="0.105565 -0.1918 -0.74405" rpy="0 0 0"/>
         <geometry>
-          <mesh filename="file:////home/cem/colcon_ws/src/Universal_Robots_ROS2_Description/meshes/ur10e/visual/shoulder.stl" scale="0.001 0.001 0.001"/>
+          <mesh filename="file:////home/emirhan/colcon_ws/src/Universal_Robots_ROS2_Description/meshes/ur10e/visual/shoulder.stl" scale="0.001 0.001 0.001"/>
         </geometry>
         <material name="silver"/>
@@ -164,5 +166,5 @@
         <origin xyz="0.105565 -0.1918 -0.74405" rpy="0 0 0"/>
         <geometry>
-          <mesh filename="file:////home/cem/colcon_ws/src/Universal_Robots_ROS2_Description/meshes/ur10e/collision/shoulder.stl" scale="0.001 0.001 0.001"/>
+          <mesh filename="file:////home/emirhan/colcon_ws/src/Universal_Robots_ROS2_Description/meshes/ur10e/collision/shoulder.stl" scale="0.001 0.001 0.001"/>
         </geometry>
       </collision>
@@ -184,5 +186,5 @@
         <origin xyz="0.105565 -0.2778 -0.83405" rpy="0 0 0"/>
         <geometry>
-          <mesh filename="file:////home/cem/colcon_ws/src/Universal_Robots_ROS2_Description/meshes/ur10e/visual/upperarm.stl" scale="0.001 0.001 0.001"/>
+          <mesh filename="file:////home/emirhan/colcon_ws/src/Universal_Robots_ROS2_Description/meshes/ur10e/visual/upperarm.stl" scale="0.001 0.001 0.001"/>
         </geometry>
         <material name="silver"/>
@@ -191,5 +193,5 @@
         <origin xyz="0.105565 -0.2778 -0.83405" rpy="0 0 0"/>
         <geometry>
-          <mesh filename="file:////home/cem/colcon_ws/src/Universal_Robots_ROS2_Description/meshes/ur10e/collision/upperarm.stl" scale="0.001 0.001 0.001"/>
+          <mesh filename="file:////home/emirhan/colcon_ws/src/Universal_Robots_ROS2_Description/meshes/ur10e/collision/upperarm.stl" scale="0.001 0.001 0.001"/>
         </geometry>
       </collision>
@@ -211,5 +213,5 @@
         <origin xyz="-0.506534 -0.299691 -0.833449" rpy="0 0 0"/>
         <geometry>
-          <mesh filename="file:////home/cem/colcon_ws/src/Universal_Robots_ROS2_Description/meshes/ur10e/visual/forearm.stl" scale="0.001 0.001 0.001"/>
+          <mesh filename="file:////home/emirhan/colcon_ws/src/Universal_Robots_ROS2_Description/meshes/ur10e/visual/forearm.stl" scale="0.001 0.001 0.001"/>
         </geometry>
         <material name="silver"/>
@@ -218,5 +220,5 @@
         <origin xyz="-0.506534 -0.299691 -0.833449" rpy="0 0 0"/>
         <geometry>
-          <mesh filename="file:////home/cem/colcon_ws/src/Universal_Robots_ROS2_Description/meshes/ur10e/collision/forearm.stl" scale="0.001 0.001 0.001"/>
+          <mesh filename="file:////home/emirhan/colcon_ws/src/Universal_Robots_ROS2_Description/meshes/ur10e/collision/forearm.stl" scale="0.001 0.001 0.001"/>
         </geometry>
       </collision>
@@ -238,5 +240,5 @@
       	<origin xyz="-1.078132 -0.301691 -0.833449" rpy="0 0 0"/>
         <geometry>
-          <mesh filename="file:////home/cem/colcon_ws/src/Universal_Robots_ROS2_Description/meshes/ur10e/visual/wrist1.stl" scale="0.001 0.001 0.001"/>
+          <mesh filename="file:////home/emirhan/colcon_ws/src/Universal_Robots_ROS2_Description/meshes/ur10e/visual/wrist1.stl" scale="0.001 0.001 0.001"/>
         </geometry>
         <material name="silver"/>
@@ -245,5 +247,5 @@
         <origin xyz="-1.078132 -0.301691 -0.833449" rpy="0 0 0"/>
         <geometry>
-          <mesh filename="file:////home/cem/colcon_ws/src/Universal_Robots_ROS2_Description/meshes/ur10e/collision/wrist1.stl" scale="0.001 0.001 0.001"/>
+          <mesh filename="file:////home/emirhan/colcon_ws/src/Universal_Robots_ROS2_Description/meshes/ur10e/collision/wrist1.stl" scale="0.001 0.001 0.001"/>
         </geometry>
       </collision>
@@ -265,5 +267,5 @@
         <origin xyz="-1.078132 -0.355691 -0.77175" rpy="0 0 0"/>
         <geometry>
-          <mesh filename="file:////home/cem/colcon_ws/src/Universal_Robots_ROS2_Description/meshes/ur10e/visual/wrist2.stl" scale="0.001 0.001 0.001"/>
+          <mesh filename="file:////home/emirhan/colcon_ws/src/Universal_Robots_ROS2_Description/meshes/ur10e/visual/wrist2.stl" scale="0.001 0.001 0.001"/>
         </geometry>
         <material name="silver"/>
@@ -272,5 +274,5 @@
         <origin xyz="-1.078132 -0.355691 -0.77175" rpy="0 0 0"/>
         <geometry>
-          <mesh filename="file:////home/cem/colcon_ws/src/Universal_Robots_ROS2_Description/meshes/ur10e/collision/wrist2.stl" scale="0.001 0.001 0.001"/>
+          <mesh filename="file:////home/emirhan/colcon_ws/src/Universal_Robots_ROS2_Description/meshes/ur10e/collision/wrist2.stl" scale="0.001 0.001 0.001"/>
         </geometry>
       </collision>
@@ -292,5 +294,5 @@
         <origin xyz="-1.078132 -0.417389 -0.71775" rpy="0 0 0"/>
         <geometry>
-          <mesh filename="file:////home/cem/colcon_ws/src/Universal_Robots_ROS2_Description/meshes/ur10e/visual/wrist3.stl" scale="0.001 0.001 0.001"/>
+          <mesh filename="file:////home/emirhan/colcon_ws/src/Universal_Robots_ROS2_Description/meshes/ur10e/visual/wrist3.stl" scale="0.001 0.001 0.001"/>
         </geometry>
         <material name="silver"/>
@@ -299,5 +301,5 @@
         <origin xyz="-1.078132 -0.417389 -0.71775" rpy="0 0 0"/>
         <geometry>
-          <mesh filename="file:////home/cem/colcon_ws/src/Universal_Robots_ROS2_Description/meshes/ur10e/collision/wrist3.stl" scale="0.001 0.001 0.001"/>
+          <mesh filename="file:////home/emirhan/colcon_ws/src/Universal_Robots_ROS2_Description/meshes/ur10e/collision/wrist3.stl" scale="0.001 0.001 0.001"/>
         </geometry>
       </collision>
@@ -440,5 +442,5 @@
         <origin xyz="-1.106132 -0.502789 -0.727752" rpy="0 0 0"/>
         <geometry>
-          <mesh filename="file:////home/cem/colcon_ws/src/Universal_Robots_ROS2_Description/meshes/ur10e/collision/flange.stl" scale="0.001 0.001 0.001"/>
+          <mesh filename="file:////home/emirhan/colcon_ws/src/Universal_Robots_ROS2_Description/meshes/ur10e/collision/flange.stl" scale="0.001 0.001 0.001"/>
         </geometry>
         <material name="silver"/>
@@ -447,5 +449,5 @@
         <origin xyz="-1.106132 -0.502789 -0.727752" rpy="0 0 0"/>
         <geometry>
-          <mesh filename="file:////home/cem/colcon_ws/src/Universal_Robots_ROS2_Description/meshes/ur10e/collision/flange.stl" scale="0.001 0.001 0.001"/>
+          <mesh filename="file:////home/emirhan/colcon_ws/src/Universal_Robots_ROS2_Description/meshes/ur10e/collision/flange.stl" scale="0.001 0.001 0.001"/>
         </geometry>
       </collision>
@@ -466,5 +468,5 @@
         <origin xyz="-1.078132 -0.477889 -0.717752" rpy="0 0 0"/>
         <geometry>
-          <mesh filename="file:////home/cem/colcon_ws/src/Universal_Robots_ROS2_Description/meshes/ur10e/collision/tool0.stl" scale="0.001 0.001 0.001"/>
+          <mesh filename="file:////home/emirhan/colcon_ws/src/Universal_Robots_ROS2_Description/meshes/ur10e/collision/tool0.stl" scale="0.001 0.001 0.001"/>
         </geometry>
         <material name="silver"/>
@@ -473,5 +475,5 @@
         <origin xyz="-1.078132 -0.477889 -0.717752" rpy="0 0 0"/>
         <geometry>
-          <mesh filename="file:////home/cem/colcon_ws/src/Universal_Robots_ROS2_Description/meshes/ur10e/collision/tool0.stl" scale="0.001 0.001 0.001"/>
+          <mesh filename="file:////home/emirhan/colcon_ws/src/Universal_Robots_ROS2_Description/meshes/ur10e/collision/tool0.stl" scale="0.001 0.001 0.001"/>
         </geometry>
       </collision>
@@ -486,5 +488,5 @@
         <origin xyz="-1.02433 -0.5466 -0.730752" rpy="0 0 0"/>
         <geometry>
-          <mesh filename="file:////home/cem/colcon_ws/src/Universal_Robots_ROS2_Description/meshes/ur10e/collision/sick_camera_mo.stl" scale="0.001 0.001 0.001"/>
+          <mesh filename="file:////home/emirhan/colcon_ws/src/Universal_Robots_ROS2_Description/meshes/ur10e/collision/sick_camera_mo.stl" scale="0.001 0.001 0.001"/>
         </geometry>
         <material name="silver"/>
@@ -493,5 +495,5 @@
         <origin xyz="-1.02433 -0.5466 -0.730752" rpy="0 0 0"/>
         <geometry>
-          <mesh filename="file:////home/cem/colcon_ws/src/Universal_Robots_ROS2_Description/meshes/ur10e/collision/sick_camera_mo.stl" scale="0.001 0.001 0.001"/>
+          <mesh filename="file:////home/emirhan/colcon_ws/src/Universal_Robots_ROS2_Description/meshes/ur10e/collision/sick_camera_mo.stl" scale="0.001 0.001 0.001"/>
         </geometry>
       </collision>
@@ -506,5 +508,5 @@
         <origin xyz="-1.078132 -0.537789 -0.707752" rpy="0 0 0"/>
         <geometry>
-          <mesh filename="file:////home/cem/colcon_ws/src/Universal_Robots_ROS2_Description/meshes/ur10e/collision/cable_channel_flange.stl" scale="0.001 0.001 0.001"/>
+          <mesh filename="file:////home/emirhan/colcon_ws/src/Universal_Robots_ROS2_Description/meshes/ur10e/collision/cable_channel_flange.stl" scale="0.001 0.001 0.001"/>
         </geometry>
         <material name="silver"/>
@@ -513,5 +515,5 @@
         <origin xyz="-1.078132 -0.537789 -0.707752" rpy="0 0 0"/>
         <geometry>
-          <mesh filename="file:////home/cem/colcon_ws/src/Universal_Robots_ROS2_Description/meshes/ur10e/collision/cable_channel_flange.stl" scale="0.001 0.001 0.001"/>
+          <mesh filename="file:////home/emirhan/colcon_ws/src/Universal_Robots_ROS2_Description/meshes/ur10e/collision/cable_channel_flange.stl" scale="0.001 0.001 0.001"/>
         </geometry>
       </collision>
@@ -526,5 +528,5 @@
         <origin xyz="-1.078132 -0.486789 -0.669752" rpy="0 0 0"/>
         <geometry>
-          <mesh filename="file:////home/cem/colcon_ws/src/Universal_Robots_ROS2_Description/meshes/ur10e/collision/cable_channel.stl" scale="0.001 0.001 0.001"/>
+          <mesh filename="file:////home/emirhan/colcon_ws/src/Universal_Robots_ROS2_Description/meshes/ur10e/collision/cable_channel.stl" scale="0.001 0.001 0.001"/>
         </geometry>
         <material name="silver"/>
@@ -533,5 +535,5 @@
         <origin xyz="-1.078132 -0.486789 -0.669752" rpy="0 0 0"/>
         <geometry>
-          <mesh filename="file:////home/cem/colcon_ws/src/Universal_Robots_ROS2_Description/meshes/ur10e/collision/cable_channel.stl" scale="0.001 0.001 0.001"/>
+          <mesh filename="file:////home/emirhan/colcon_ws/src/Universal_Robots_ROS2_Description/meshes/ur10e/collision/cable_channel.stl" scale="0.001 0.001 0.001"/>
         </geometry>
       </collision>
@@ -581,4 +583,154 @@
       <child link="${tf_prefix}rgb_optical_frame"/>
     </joint>
+    <xacro:if value="${use_gripper}">
+      <link name="${tf_prefix}gripper_body_1">
+        <inertial>
+          <origin xyz="0.046201794305521515 0.04641351769017876 -0.017675503740650633" rpy="0 0 0"/>
+          <mass value="4.92893092862587"/>
+          <inertia ixx="0.006626" iyy="0.0075" izz="0.005595" ixy="-0.000805" iyz="4e-06" ixz="8e-06"/>
+        </inertial>
+        <visual>
+          <origin xyz="-1.123708 -0.518786 -0.735428" rpy="0 0 0"/>
+          <geometry>
+            <mesh filename="file:////home/emirhan/colcon_ws/src/Universal_Robots_ROS2_Description/meshes/ur10e/secondrobotcollision/gripper_body_1.stl" scale="0.001 0.001 0.001"/>
+          </geometry>
+          <material name="violet">
+            <color rgba="0.4 0.18 0.57 1.0"/>
+          </material>
+        </visual>
+        <collision>
+          <origin xyz="-1.123708 -0.518786 -0.735428" rpy="0 0 0"/>
+          <geometry>
+            <mesh filename="file:////home/emirhan/colcon_ws/src/Universal_Robots_ROS2_Description/meshes/ur10e/secondrobotcollision/gripper_body_1.stl" scale="0.001 0.001 0.001"/>
+          </geometry>
+        </collision>
+      </link>
+      <link name="${tf_prefix}gripper_upper_1">
+        <inertial>
+          <origin xyz="0.009933945618336715 0.020191952923398593 0.002410109555269213" rpy="0 0 0"/>
+          <mass value="0.15599517357950826"/>
+          <inertia ixx="3.7e-05" iyy="4.5e-05" izz="6.6e-05" ixy="-7e-06" iyz="-5e-06" ixz="-9e-06"/>
+        </inertial>
+        <visual>
+          <origin xyz="-1.22001 -0.579787 -0.7675" rpy="0 0 0"/>
+          <geometry>
+            <mesh filename="file:////home/emirhan/colcon_ws/src/Universal_Robots_ROS2_Description/meshes/ur10e/secondrobotcollision/gripper_upper_1.stl" scale="0.001 0.001 0.001"/>
+          </geometry>
+          <material name="grey">
+            <color rgba="0.2 0.2 0.2 1.0"/>
+          </material>
+        </visual>
+        <collision>
+          <origin xyz="-1.22001 -0.579787 -0.7675" rpy="0 0 0"/>
+          <geometry>
+            <mesh filename="file:////home/emirhan/colcon_ws/src/Universal_Robots_ROS2_Description/meshes/ur10e/secondrobotcollision/gripper_upper_1.stl" scale="0.001 0.001 0.001"/>
+          </geometry>
+        </collision>
+      </link>
+      <link name="${tf_prefix}gripper_lower_1">
+        <inertial>
+          <origin xyz="0.009953097781983722 0.020157371452492412 -0.0024101337743568374" rpy="0 0 0"/>
+          <mass value="0.15599517357965467"/>
+          <inertia ixx="3.7e-05" iyy="4.5e-05" izz="6.6e-05" ixy="-7e-06" iyz="5e-06" ixz="9e-06"/>
+        </inertial>
+        <visual>
+          <origin xyz="-1.22001 -0.579787 -0.668" rpy="0 0 0"/>
+          <geometry>
+            <mesh filename="file:////home/emirhan/colcon_ws/src/Universal_Robots_ROS2_Description/meshes/ur10e/secondrobotcollision/gripper_lower_1.stl" scale="0.001 0.001 0.001"/>
+          </geometry>
+          <material name="grey">
+            <color rgba="0.2 0.2 0.2 1.0"/>
+          </material>
+        </visual>
+        <collision>
+          <origin xyz="-1.22001 -0.579787 -0.668" rpy="0 0 0"/>
+          <geometry>
+            <mesh filename="file:////home/emirhan/colcon_ws/src/Universal_Robots_ROS2_Description/meshes/ur10e/secondrobotcollision/gripper_lower_1.stl" scale="0.001 0.001 0.001"/>
+          </geometry>
+        </collision>
+      </link>
+      <joint name="${tf_prefix}gripper_body_joint" type="fixed">
+        <origin xyz="0.045576 0.040897 0.017678" rpy="0 0 0"/>
+        <parent link="${tf_prefix}tool0"/>
+        <child link="${tf_prefix}gripper_body_1"/>
+      </joint>
+      <joint name="${tf_prefix}gripper_joint" type="prismatic">
+        <origin xyz="0.096302 0.061001 0.032072" rpy="0 0 0"/>
+        <parent link="${tf_prefix}gripper_body_1"/>
+        <child link="${tf_prefix}gripper_upper_1"/>
+        <axis xyz="0.0 0.0 -1.0"/>
+        <!-- limits extended ±0.001 beyond nominal 0..0.025 range to work around DART servo bug (dartsim/dart#1683) -->
+        <limit upper="0.026" lower="-0.001" effort="1000" velocity="10"/>
+      </joint>
+      <joint name="${tf_prefix}gripper_lower_finger_joint" type="prismatic">
+        <origin xyz="0.096302 0.061001 -0.067428" rpy="0 0 0"/>
+        <parent link="${tf_prefix}gripper_body_1"/>
+        <child link="${tf_prefix}gripper_lower_1"/>
+        <axis xyz="0.0 0.0 -1.0"/>
+        <mimic joint="${tf_prefix}gripper_joint" multiplier="-1.0"/>
+        <!-- limits extended ±0.001 beyond nominal -0.025..0 range to work around DART servo bug (dartsim/dart#1683) -->
+        <limit upper="0.001" lower="-0.026" effort="1000" velocity="10"/>
+      </joint>
+      <link name="${tf_prefix}IMX_Camera">
+        <inertial>
+          <origin xyz="-3.465374807465338e-05 0.0003801084631929186 0.006566275485619721" rpy="0 0 0"/>
+          <mass value="0.04632955033200952"/>
+          <inertia ixx="5e-06" iyy="5e-06" izz="6e-06" ixy="-0.0" iyz="0.0" ixz="-0.0"/>
+        </inertial>
+        <visual>
+          <origin xyz="-0.965545 -0.534467 -0.764722" rpy="0 0 0"/>
+          <geometry>
+            <mesh filename="file:////home/emirhan/colcon_ws/src/Universal_Robots_ROS2_Description/meshes/ur10e/secondrobotcollision/IMX_Camera.stl" scale="0.001 0.001 0.001"/>
+          </geometry>
+          <material name="silver"/>
+        </visual>
+        <collision>
+          <origin xyz="-0.965545 -0.534467 -0.764722" rpy="0 0 0"/>
+          <geometry>
+            <mesh filename="file:////home/emirhan/colcon_ws/src/Universal_Robots_ROS2_Description/meshes/ur10e/secondrobotcollision/IMX_Camera.stl" scale="0.001 0.001 0.001"/>
+          </geometry>
+        </collision>
+      </link>
+      <joint name="${tf_prefix}IMX_Camera_joint" type="fixed">
+        <origin xyz="-0.058785 -0.012133 0.033972" rpy="0 0 0"/>
+        <parent link="${tf_prefix}sick_camera"/>
+        <child link="${tf_prefix}IMX_Camera"/>
+      </joint>
+      <link name="${tf_prefix}IMX_Camera_frame_link"/>
+      <joint name="${tf_prefix}IMX_Camera_frame_joint" type="fixed">
+        <!-- Datasheet: toplam derinlik 24.68mm, optik merkez lensin önünde -->
+        <origin xyz="0.0 0.025 0.0" rpy="0 0 0" />
+        <parent link="${tf_prefix}IMX_Camera" />
+        <child link="${tf_prefix}IMX_Camera_frame_link"/>
+      </joint>
+      <link name="${tf_prefix}IMX_optical_frame"/>
+      <joint name="${tf_prefix}IMX_optical_joint" type="fixed">
+        <origin xyz="0 0 0" rpy="0 0 ${M_PI/2}" />
+        <parent link="${tf_prefix}IMX_Camera_frame_link" />
+        <child link="${tf_prefix}IMX_optical_frame"/>
+      </joint>
+      <gazebo reference="${tf_prefix}IMX_Camera_frame_link">
+        <sensor name="${tf_prefix}imx179_camera" type="camera">
+          <!-- +Z yönüne bak (roll=-π/2) -->
+          <pose>0 0 0 0 -1.5708 0</pose>
+          <always_on>true</always_on>
+          <update_rate>30.0</update_rate>
+          <visualize>false</visualize>
+          <camera name="${tf_prefix}imx179_rgb">
+            <!-- 145 deg = 2.5307 rad -->
+            <horizontal_fov>2.5307</horizontal_fov>
+            <image>
+              <width>1920</width>
+              <height>1080</height>
+              <format>R8G8B8</format>
+            </image>
+            <clip>
+              <near>0.05</near>
+              <far>16.0</far>
+            </clip>
+          </camera>
+        </sensor>
+      </gazebo>
+    </xacro:if>
   </xacro:macro>
 </robot>
