Commit message: 2fg7

File: onrobot_2fg7_description/ros2_control/onrobot_2fg7.ros2_control.xacro (robot description, xacro)
@@ -18,5 +18,5 @@
         </xacro:if>
       </hardware>
-      <joint name="${prefix}ur10e_gripper_joint">
+      <joint name="${prefix}gripper_joint">
         <state_interface name="position"/>
         <state_interface name="velocity"/>

File: onrobot_2fg7_description/urdf/materials.xacro (robot description, xacro)
@@ -1,6 +1,6 @@
 <?xml version="1.0" ?>
 <robot name="2FG7_outwards" xmlns:xacro="http://www.ros.org/wiki/xacro" >
-<material name="silver">
+<!-- <material name="silver">
   <color rgba="0.700 0.700 0.700 1.000"/>
-</material>
+</material> -->
 </robot>

File: onrobot_2fg7_description/urdf/onrobot_2fg7.urdf.xacro (robot description, xacro)
@@ -7,8 +7,8 @@
     <xacro:arg name="velocity_filtering" default="" />
     <xacro:arg name="use_mock_hardware" default="false"/>
-    <xacro:include filename="$(find ur_description)/urdf/ur_macro.xacro"/>
+    <!-- <xacro:include filename="$(find ur_description)/urdf/ur_macro.xacro"/> -->
     <xacro:include filename="$(find onrobot_2fg7_description)/urdf/onrobot_2fg7.xacro"/>
     <xacro:include filename="$(find onrobot_2fg7_description)/ros2_control/onrobot_2fg7.ros2_control.xacro"/>
-    <link name="world"></link>
+    <!-- <link name="world"></link>
     <xacro:ur_robot
         name="ur10e"
@@ -23,5 +23,5 @@
         sim_ignition="false">
         <origin xyz="0 0 0" rpy="0 0 0"/>
-    </xacro:ur_robot>
+    </xacro:ur_robot> -->
     <xacro:onrobot_2fg7 prefix="$(arg prefix)" parent="ur_tool0">
         <origin xyz="0.045576 0.040897 0.017678" rpy="0 0 0"/>

File: onrobot_2fg7_description/urdf/onrobot_2fg7.xacro (robot description, xacro)
@@ -4,5 +4,5 @@
   <xacro:include filename="$(find onrobot_2fg7_description)/urdf/materials.xacro" />
   <xacro:macro name="onrobot_2fg7" params="prefix parent *origin">
-    <link name="${prefix}base_link">
+    <link name="${prefix}gripper_base_link">
       <inertial>
         <origin xyz="0.046201794305521515 0.04641351769017876 -0.017675503740650633" rpy="0 0 0"/>
@@ -26,5 +26,5 @@
       </collision>
     </link>
-    <link name="${prefix}ur10e_gripper_upper_1">
+    <link name="${prefix}gripper_upper_1">
       <inertial>
         <origin xyz="0.009933945618336715 0.020191952923398593 0.002410109555269213" rpy="0 0 0"/>
@@ -48,5 +48,5 @@
       </collision>
     </link>
-    <link name="${prefix}ur10e_gripper_lower_1">
+    <link name="${prefix}gripper_lower_1">
       <inertial>
         <origin xyz="0.009953097781983722 0.020157371452492412 -0.0024101337743568374" rpy="0 0 0"/>
@@ -70,24 +70,24 @@
       </collision>
     </link>
-    <joint name="${prefix}ur10e_gripper_joint" type="prismatic">
+    <joint name="${prefix}gripper_joint" type="prismatic">
       <origin xyz="0.096302 0.061001 0.032072" rpy="0 0 0"/>
-      <parent link="${prefix}base_link"/>
-      <child link="${prefix}ur10e_gripper_upper_1"/>
+      <parent link="${prefix}gripper_base_link"/>
+      <child link="${prefix}gripper_upper_1"/>
       <axis xyz="0.0 0.0 -1.0"/>
       <!-- limits extended ±0.001 beyond nominal 0..0.025 range to work around DART servo bug -->
       <limit upper="0.026" lower="-0.001" effort="1000" velocity="10"/>
     </joint>
-    <joint name="${prefix}ur10e_right_finger_joint" type="prismatic">
+    <joint name="${prefix}right_finger_joint" type="prismatic">
       <origin xyz="0.096302 0.061001 -0.067428" rpy="0 0 0"/>
-      <parent link="${prefix}base_link"/>
-      <child link="${prefix}ur10e_gripper_lower_1"/>
+      <parent link="${prefix}gripper_base_link"/>
+      <child link="${prefix}gripper_lower_1"/>
       <axis xyz="0.0 0.0 -1.0"/>
-      <mimic joint="${prefix}ur10e_gripper_joint" multiplier="-1.0"/>
+      <mimic joint="${prefix}gripper_joint" multiplier="-1.0"/>
       <!-- limits extended ±0.001 beyond nominal -0.025..0 range to work around DART servo bug -->
       <limit upper="0.001" lower="-0.026" effort="1000" velocity="10"/>
     </joint>
-    <joint name="${prefix}ur10e_2fg7_attach_joint" type="fixed">
+    <joint name="${prefix}2fg7_attach_joint" type="fixed">
       <parent link="${parent}"/>
-      <child link="${prefix}base_link"/>
+      <child link="${prefix}gripper_base_link"/>
       <xacro:insert_block name="origin"/>
       <axis xyz="0 0 1"/>
